Commit message: add instructions for implementing slam

File: description/robot_core.xacro (robot description, xacro)
@@ -18,4 +18,7 @@
     </link>
     <!-- BASE_FOOTPRINT LINK -->
+    <link name="base_footprint">
+    </link>
+    <!-- BASE_FOOTPRINT LINK -->
     <joint name="base_footprint_joint" type="fixed">
         <parent link="base_link"/>
@@ -23,6 +26,4 @@
         <origin xyz="0 0 0" rpy="0 0 0"/>
     </joint>
-    <link name="base_footprint">
-    </link>
     <!-- CHASSIS LINK -->
     <joint name="chassis_joint" type="fixed">
